File: kicad/main_board.kicad_sch (KiCad schematic)
At the start: 65 parts, among them J1 Conn_01x18, J2 Conn_01x18, J3 Conn_01x07, J4 Conn_01x07, J5 Conn_01x07, J6 Conn_01x07, J7 Conn_01x07, J8 TYPE-C-31-M-12, J9 TYPE-C-31-M-12, Q1 DMG2301L-7, Q2 DMG2301L-7, Q3 DMG2301L-7, Q4 DMG2301L-7, Q5 DMG2301L-7, SW1 Reset, SW2 Boot, U1 XC6220B331MR, U2 RP2040, U3 W25Q128JVS, U4 COS724, U5 COS724, U6 USBLC6-2SC6, U7 USBLC6-2SC6, Y1 Crystal_GND24

Commit message: Modifications to additional headers
- Added mouse header
- Added additional columns to support thumb through
- Switched to ribbon cables
Parts:
- removed unit 4 of U5
- added R18: 2k, Resistor_SMD:R_0402_1005Metric_Pad0.72x0.64mm_HandSolder, symbol Device:R_Small
- added unit 1 of U5
- added U8, U9: FPC-0.5FX-6PWCR-H20, easyeda2kicad:FPC-SMD_6P-P0.50_FPC-0.5FX-6PWCR-H20, symbol easyeda2kicad:FPC-0.5FX-6PWCR-H20
- J3, J4, J5, J6, J7: footprint lalboard:JST_ZH_B7B-ZR_1x07_P1.50mm_Vertical -> easyeda2kicad:FPC-SMD_8P-P0.50_AFC11-S08ICC-00; symbol Connector_Generic:Conn_01x07 -> Connector_Generic:Conn_01x08; now in the parts list
Connections:
- net +3.3V: now also U8.1, U9.1
- net AMP_REF: now also U5.10 (+), U5.12 (+), U5.5 (+), U5.3 (+); no longer U5.10 (+), U5.3 (+), U5.5 (+)
- net COL1: now also J3.7 (Pin_7), J4.7 (Pin_7), J5.7 (Pin_7), J6.7 (Pin_7), J7.7 (Pin_7); no longer J3.6 (Pin_6), J4.6 (Pin_6), J5.6 (Pin_6), J6.6 (Pin_6), J7.6 (Pin_6)
- net COL2: now also J3.6 (Pin_6), J4.6 (Pin_6), J5.6 (Pin_6), J6.6 (Pin_6), J7.6 (Pin_6); no longer J3.5 (Pin_5), J4.5 (Pin_5), J5.5 (Pin_5), J6.5 (Pin_5), J7.5 (Pin_5)
- net COL3: now also J3.5 (Pin_5), J4.5 (Pin_5), J5.5 (Pin_5), J6.5 (Pin_5), J7.5 (Pin_5); no longer J3.4 (Pin_4), J4.4 (Pin_4), J5.4 (Pin_4), J6.4 (Pin_4), J7.4 (Pin_4)
- net COL4: now also J3.4 (Pin_4), J4.4 (Pin_4), J5.4 (Pin_4), J6.4 (Pin_4), J7.4 (Pin_4), U5.9 (-); no longer J3.3 (Pin_3), J4.3 (Pin_3), J5.3 (Pin_3), J6.3 (Pin_3), J7.3 (Pin_3), U5.6 (-)
- net COL4_AMP: now also U5.8; no longer U5.7
- net COL5: now also J3.3 (Pin_3), J4.3 (Pin_3), J5.3 (Pin_3), J6.3 (Pin_3), J7.3 (Pin_3), U5.13 (-); no longer J3.2 (Pin_2), J4.2 (Pin_2), J5.2 (Pin_2), J6.2 (Pin_2), J7.2 (Pin_2), U5.2 (-)
- net COL5_AMP: now also U5.14; no longer U5.1
- net GND: now also U8.6, U9.6
- net at Q3.2 (S): now also J5.8 (Pin_8); no longer J5.7 (Pin_7)
- net at Q2.2 (S): now also J4.8 (Pin_8); no longer J4.7 (Pin_7)
- net at Q1.2 (S): now also J3.8 (Pin_8); no longer J3.7 (Pin_7)
- net at Q5.2 (S): now also J7.8 (Pin_8); no longer J7.7 (Pin_7)
- net at Q4.2 (S): now also J6.8 (Pin_8); no longer J6.7 (Pin_7)
- net GPIO10 renamed SCK1
- net SCK1: now also U8.4
- net GPIO11 renamed MOSI1
- net MOSI1: now also U8.3
- net GPIO12 renamed SS1
- net SS1: now also U8.2
- net GPIO13 renamed COL6_AMP
- net COL6_AMP: now also R18.1, U5.1
- net GPIO5 renamed MISO2
- net MISO2: now also U9.5
- net GPIO6 renamed SCK2
- net SCK2: now also U9.4
- net GPIO7 renamed MOSI2
- net MOSI2: now also U9.3
- net GPIO8 renamed SS2
- net SS2: now also U9.2
- net GPIO9 renamed MISO1
- net MISO1: now also U8.5
- new net: U5.6 (-), U5.7
- new net COL6: J3.2 (Pin_2), J4.2 (Pin_2), J5.2 (Pin_2), J6.2 (Pin_2), J7.2 (Pin_2), R18.2, U5.2 (-)
Other:
- note added: "Track Balls"
- note added: "https://github.com/Bastardkb/charybdis-pmw-3360-sensor-pcb"
- moved on the sheet: Q2, Q3, Q4, Q5

Commit message: Single Trackball Correction
No need for two trackballs per side.
Parts:
- removed U9: FPC-0.5FX-6PWCR-H20, easyeda2kicad:FPC-SMD_6P-P0.50_FPC-0.5FX-6PWCR-H20, symbol easyeda2kicad:FPC-0.5FX-6PWCR-H20
Connections:
- net MISO2 renamed GPIO5
- net MOSI2 renamed GPIO7
- net SCK2 renamed GPIO6
- net SS2 renamed GPIO8
Other:
- note added: "Track Ball"
- note removed: "Track Balls"
