File: kicad/thumb_cluster_right.kicad_sch (KiCad schematic)
At the start: 18 parts, among them J1 Conn_01x07

Commit message: Initial commit of lalboard extended features, including breakout board.
Parts:
- added SW1: TS-1187A-B-A-B, easyeda2kicad:SW-SMD_4P-L5.1-W5.1-P3.70-LS6.5-TL_H1.5, symbol easyeda2kicad:TS-1187A-B-A-B
- added U1: WS2812D-255, easyeda2kicad:LED-TH_4P-L5.0-W2.5-P1.27_WS2812D-255, symbol easyeda2kicad:WS2812D-255
- H1, H2: footprint MountingHole:MountingHole_3.2mm_M3_Pad -> MountingHole:MountingHole_2.2mm_M2_DIN965_Pad
- IR1, IR2, IR3, IR4, IR5, PT1, PT2, PT3, PT4, PT5, R1, R2, R3, R4, R5: now not fitted
- J1: footprint lalboard:JST_ZH_B7B-ZR_1x07_P1.50mm_Vertical -> Connector_Wuerth:Wuerth_WR-WTB_64801011622_1x10_P1.50mm_Vertical; symbol Connector_Generic:Conn_01x07 -> Connector_Generic:Conn_01x10
Connections:
- net +3.3V: now also J1.4 (Pin_4); no longer J1.1 (Pin_1)
- net C1: now also J1.5 (Pin_5); no longer J1.2 (Pin_2)
- net C2: now also J1.6 (Pin_6); no longer J1.3 (Pin_3)
- net C3: now also J1.7 (Pin_7); no longer J1.4 (Pin_4)
- net C4: now also J1.8 (Pin_8); no longer J1.5 (Pin_5)
- net C5: now also J1.9 (Pin_9); no longer J1.6 (Pin_6)
- net GND: now also J1.10 (Pin_10), SW1.3 (C), SW1.4 (D), U1.3 (CATHODE); no longer J1.7 (Pin_7)
- new net +5V: J1.1 (Pin_1), U1.2 (ANODE)
- new net C6: J1.3 (Pin_3), SW1.1 (A), SW1.2 (B)
- new net C7: J1.2 (Pin_2), U1.4 (DIN)
- no-connect marks 0 -> 1
